File: pcbs/proto-frl/proto-frl.kicad_pcb (KiCad board)
At the start: 2 copper layers, 349.2 x 92.1 mm, 186 parts, among them U1 W25Q128JVS, U3 RP2040, Y1 12MHz

Commit message: no i'm not dead yet and neither is the project
Parts:
- removed C12, C14 (x3), C5, C9 (x4): 100nF, Capacitor_SMD:C_0402_1005Metric
- removed C2, C3: 22pF, Capacitor_SMD:C_0402_1005Metric
- removed C4, C7: 1uF, Capacitor_SMD:C_0402_1005Metric
- removed MX_#0_1, MX_#1, MX_#2, MX_#3, MX_#4, MX_#5, MX_#6, MX_#7, MX_#8, MX_#9, MX_'1, MX_,1, MX_-1, MX_.1, MX_/1, MX_/2, MX_;1, MX_=1, MX_A1, MX_B1, MX_BACK2, MX_BACK3, MX_C1, MX_D1, MX_DEL1, MX_DN1, MX_E1, MX_END1, MX_F1, MX_G1, MX_H1, MX_HOME1, MX_I1, MX_INS1, MX_J1, MX_K1, MX_L1, MX_LFT1, MX_M1, MX_N1, MX_O1, MX_P1, MX_PGDN1, MX_PGUP1, MX_Q1, MX_R1, MX_RGUI2, MX_RSHIFT3, MX_RT1, MX_S1, MX_T1, MX_U1, MX_UP1, MX_V1, MX_W1, MX_X1, MX_Y1, MX_Z1, MX_[1, MX_\2, MX_]1, MX_`1: 1U, MX_Alps:MX-1U-NoLED
- removed MX_BACK1: 2U, MX_Alps:MX-2U-NoLED
- removed MX_CLOCK1, MX_RSHIFT2, MX_RSHIFT4: 1.75U, MX_Alps:MX-1.75U-NoLED
- removed MX_CLOCK2: MX-1.25U, MX_Alps:MX-1.25U-NoLED
- removed MX_CLOCK3: MX-1.25U, Alps_Only:ALPS-1.5U
- removed MX_LALT2, MX_LALT3, MX_LCTRL2: MX-1.5U, MX_Alps:MX-1.5U-NoLED
- removed MX_LALT4: MX-1.5U, MX_Alps:MX-1.25U-NoLED
- removed MX_LALT5: MX-1.5U, MX_Alps:MX-3U-ReversedStabilizers-NoLED
- removed MX_LGUI2: MX-1U, MX_Alps:MX-1U-NoLED
- removed MX_LGUI3: MX-1U, MX_Alps:MX-1.25U-NoLED
- removed MX_LSHIFT1: 2.25U, MX_Alps:MX-2.25U-ReversedStabilizers-NoLED
- removed MX_RALT2, MX_RALT3, MX_RALT4, MX_RCTRL2, MX_TAB1, MX_\1: 1.5U, MX_Alps:MX-1.5U-NoLED
- removed MX_RALT5: 1.5U, MX_Alps:MX-1.25U-NoLED
- removed MX_RETURN1: 2.25U, MX_Alps:MX-2.25U-NoLED
- removed MX_RETURN2: MX-ISO, MX_Alps_Hybrid:MX-ISO-ReversedStabilizers
- removed MX_RGUI3: 1U, MX_Alps:MX-1.25U-NoLED
- removed MX_RSHIFT1: 2.75U, MX_Alps:MX-2.75U-ReversedStabilizers-NoLED
- removed MX_SP1 (x2): MX-7U, MX_Alps:MX-7U-ReversedStabilizers-NoLED
- removed MX_SP2: MX-7U, MX_Alps:MX-10U-ReversedStabilizers-NoLED
- removed MX_SP3: MX-7U, MX_Alps:MX-6.5U-ReversedStabilizers-NoLED
- removed R5, R6: 27R, Resistor_SMD:R_0603_1608Metric
- removed R7: 1k, Resistor_SMD:R_0402_1005Metric
- removed REF**0, REF**100, REF**101, REF**102, REF**103, REF**104, REF**80, REF**81, REF**82, REF**83, REF**84, REF**85, REF**86, REF**87, REF**88, REF**89, REF**90, REF**91, REF**92, REF**93, REF**94, REF**95, REF**96, REF**97, REF**98, REF**99: D_SOD-123-Pretty, random-keyboard-parts:D_SOD-123-Pretty
- removed the REF**13 at (156.8, 148.9)
- removed the REF**13 at (164.0, 129.9)
- removed the REF**13 at (159.2, 110.8)
- removed the REF**13 at (156.8, 91.8)
- removed the REF**29 at (242.6, 110.8)
- removed the REF**30 at (261.6, 110.8)
- removed the REF**42 at (290.2, 129.9)
- removed the REF**44 at (328.3, 129.9)
- removed U1: W25Q128JVS, Package_SO:SOIC-8_5.23x5.23mm_P1.27mm
- removed U3: RP2040, Sleep-Lib:RP2040-QFN-56
- removed Y1: 12MHz, Crystal:Crystal_SMD_3225-4Pin_3.2x2.5mm
- added Q1: TIP120, Package_TO_SOT_THT:TO-220-3_Vertical, B.Cu at (349.9, 66.0)
- added Q1: TIP120, Package_TO_SOT_THT:TO-220-3_Vertical, B.Cu at (355.0, 71.1)
- added REF**: 1U, MX_Alps:MX-1U-NoLED, F.Cu at (38.1, 38.1)
- added REF**: ISO-Combined, MX_Alps:MX-ISO-ReversedStabilizers, F.Cu at (302.4, 66.7)
- added REF**: Memes lol, random-keyboard-parts:Reset_Pretty, B.Cu at (317.5, 38.1)
- added REF**: D_SOD-323, Diode_SMD:D_SOD-323, B.Cu at (324.6, 38.1)
- added REF**: D_SOD-323, Diode_SMD:D_SOD-323, B.Cu at (324.6, 35.6)
- added REF**13: 1U, MX_Alps:MX-1U-NoLED, F.Cu at (285.8, 38.1)
- added REF**13: 1U, MX_Alps:MX-2U-NoLED, F.Cu at (295.3, 38.1)
- added REF**29: 1.5U, MX_Alps:MX-7U-ReversedStabilizers-NoLED, F.Cu at (171.4, 114.3)
- added REF**29: 1.5U, MX_Alps:MX-1.5U-NoLED, F.Cu at (90.5, 114.3)
- added REF**29: 1.5U, MX_Alps:MX-1.5U-NoLED, F.Cu at (42.9, 76.2)
- added REF**29: 1.5U, MX_Alps:MX-1.5U-NoLED, F.Cu at (247.7, 114.3)
- added REF**29: 1.5U, MX_Alps:MX-1.5U-NoLED, F.Cu at (223.8, 114.3)
- added REF**29: 1.25U, MX_Alps:MX-1.25U-NoLED, F.Cu at (40.5, 76.2)
- added REF**29: 1.5U, MX_Alps:MX-3U-ReversedStabilizers-NoLED, F.Cu at (157.2, 114.3)
- added REF**29: 1.5U, MX_Alps:MX-6.5U-ReversedStabilizers-NoLED, F.Cu at (171.4, 114.3)
- added REF**29: 1.5U, MX_Alps:MX-1.25U-NoLED, F.Cu at (197.6, 114.3)
- added REF**29: 1.5U, MX_Alps:MX-1.5U-NoLED, F.Cu at (95.2, 114.3)
- added REF**29: 1.5U, MX_Alps:MX-1.25U-NoLED, F.Cu at (116.7, 114.3)
- added REF**29: 1.5U, MX_Alps:MX-1.25U-NoLED, F.Cu at (226.2, 114.3)
- added REF**29: 1.5U, MX_Alps:MX-1.5U-NoLED, F.Cu at (300.0, 114.3)
- added REF**29: 1.5U, MX_Alps:MX-1.5U-NoLED, F.Cu at (42.9, 114.3)
- added REF**29: 1.25U, MX_Alps:MX-1.25U-NoLED, F.Cu at (40.5, 95.2)
- added REF**29: 1.5U, MX_Alps:MX-1.5U-NoLED, F.Cu at (252.4, 114.3)
- added REF**30: 1.75U, MX_Alps:MX-1.75U-NoLED, F.Cu at (45.2, 76.2)
- added REF**30: 1.75U, MX_Alps:MX-1.75U-NoLED, F.Cu at (278.6, 95.2)
- added REF**30: 1.75U, MX_Alps:MX-1.75U-NoLED, F.Cu at (297.7, 95.2)
- added REF**42: 2.25U, MX_Alps:MX-2.25U-NoLED, F.Cu at (292.9, 76.2)
- added REF**42: 2.25U, MX_Alps:MX-2.25U-NoLED, F.Cu at (50.0, 95.2)
- added REF**44: 1U, MX_Alps:MX-1.25U-NoLED, F.Cu at (273.8, 114.3)
- added REF**44: 1U, MX_Alps:MX-1U-NoLED, F.Cu at (276.2, 114.3)
- added REF**47: 1U, MX_Alps:MX-1U-NoLED, F.Cu at (81.0, 95.2)
- added REF**48: 1U, MX_Alps:MX-1U-NoLED, F.Cu at (100.0, 95.2)
- added REF**49: 1U, MX_Alps:MX-1U-NoLED, F.Cu at (119.1, 95.2)
- added REF**50: 1U, MX_Alps:MX-1U-NoLED, F.Cu at (138.1, 95.2)
- added REF**51: 1U, MX_Alps:MX-1U-NoLED, F.Cu at (157.2, 95.2)
- added REF**52: 1U, MX_Alps:MX-1U-NoLED, F.Cu at (176.2, 95.2)
- added REF**53: 1U, MX_Alps:MX-1U-NoLED, F.Cu at (195.3, 95.2)
- added REF**54: 1U, MX_Alps:MX-1U-NoLED, F.Cu at (214.3, 95.2)
- added REF**55: 1U, MX_Alps:MX-1U-NoLED, F.Cu at (233.4, 95.2)
- added REF**56: 1U, MX_Alps:MX-1U-NoLED, F.Cu at (252.4, 95.2)
- added REF**57: 1U, MX_Alps:MX-1U-NoLED, F.Cu at (271.5, 95.2)
- added REF**58: 1U, MX_Alps:MX-2.75U-NoLED, F.Cu at (288.1, 95.2)
- added REF**59: 1U, MX_Alps:MX-1U-NoLED, F.Cu at (61.9, 95.2)
- added REF**60: 1U, MX_Alps:MX-1U-NoLED, F.Cu at (371.5, 114.3)
- added REF**61: 1U, MX_Alps:MX-1.25U-NoLED, F.Cu at (69.1, 114.3)
- added REF**61: 1U, MX_Alps:MX-1U-NoLED, F.Cu at (66.7, 114.3)
- added REF**63: 1U, MX_Alps:MX-1U-NoLED, F.Cu at (352.4, 95.2)
- added REF**68: 1U, MX_Alps:MX-1U-NoLED, F.Cu at (333.4, 57.1)
- added REF**69: 1U, MX_Alps:MX-1U-NoLED, F.Cu at (352.4, 57.1)
- added REF**70: 1U, MX_Alps:MX-1U-NoLED, F.Cu at (371.5, 57.1)
- added REF**71: 1U, MX_Alps:MX-1U-NoLED, F.Cu at (333.4, 38.1)
- added REF**72: 1U, MX_Alps:MX-1U-NoLED, F.Cu at (352.4, 38.1)
- added REF**73: 1U, MX_Alps:MX-1U-NoLED, F.Cu at (371.5, 38.1)
- added REF**75: 1U, MX_Alps:MX-1U-NoLED, F.Cu at (304.8, 95.2)
- REF**1, REF**10, REF**11, REF**12, REF**14, REF**16, REF**17, REF**18, REF**19, REF**2, REF**20, REF**21, REF**22, REF**23, REF**24, REF**25, REF**26, REF**27, REF**3, REF**31, REF**32, REF**33, REF**34, REF**35, REF**36, REF**37, REF**38, REF**39, REF**4, REF**40, REF**41, REF**43, REF**45, REF**46, REF**5, REF**6, REF**7, REF**8, REF**9: value D_SOD-123-Pretty -> 1U; footprint random-keyboard-parts:D_SOD-123-Pretty -> MX_Alps:MX-1U-NoLED; moved to F.Cu
- REF**15, REF**28: value D_SOD-123-Pretty -> 1.5U; footprint random-keyboard-parts:D_SOD-123-Pretty -> MX_Alps:MX-1.5U-NoLED; moved to F.Cu
- moved REF**31 212.1 mm to (71.4, 76.2), turned to 0 degrees
- moved REF**32 212.1 mm to (90.5, 76.2), turned to 0 degrees
- moved REF**35 212.1 mm to (147.6, 76.2), turned to 0 degrees
- moved REF**36 212.1 mm to (166.7, 76.2), turned to 0 degrees
- moved REF**33 212.1 mm to (109.5, 76.2), turned to 0 degrees
- moved REF**34 212.1 mm to (128.6, 76.2), turned to 0 degrees
- moved REF**15 160.6 mm to (42.9, 57.1), turned to 0 degrees
- moved REF**19 156.0 mm to (123.8, 57.1), turned to 0 degrees
- moved REF**24 156.0 mm to (219.1, 57.1), turned to 0 degrees
- moved REF**17 156.0 mm to (85.7, 57.1), turned to 0 degrees
- moved REF**18 156.0 mm to (104.8, 57.1), turned to 0 degrees
- moved REF**22 156.0 mm to (181.0, 57.1), turned to 0 degrees
- moved REF**23 156.0 mm to (200.0, 57.1), turned to 0 degrees
- moved REF**16 156.0 mm to (66.7, 57.1), turned to 0 degrees
- moved REF**20 156.0 mm to (142.9, 57.1), turned to 0 degrees
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Routing:
- net (no net): track 2615.2 -> 9.58 mm
- net GND: track 98.2 -> 0.00 mm, vias 9 -> 0
- net +3V3: track 41.9 -> 0.00 mm
- net +1V1: track 28.2 -> 0.00 mm, vias 4 -> 0
- net SD3: track 18.7 -> 0.00 mm
- net QSPI_CLK: track 16.8 -> 0.00 mm
- net SD0: track 12.5 -> 0.00 mm
- net XTAL_IN: track 7.35 -> 0.00 mm
- net XTAL_0: track 7.30 -> 0.00 mm
- net D+: track 6.73 -> 0.00 mm
- net D-: track 5.35 -> 0.00 mm
- net CS: track 4.95 -> 0.00 mm
- net SD1: track 4.59 -> 0.00 mm
- net SD2: track 4.26 -> 0.00 mm
- net SWCLK: track 3.79 -> 0.00 mm
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Other:
- board size 349.2 x 92.1 mm -> 348.6 x 91.4 mm
